File: Witcher/LittleKiran.kicad_sch (KiCad schematic)
At the start: 10 parts, among them J1 XT60PW-M, J2 XT60PW-M, J3 XT60PW-M, Q1 PXP012-30QLJ, Q2 PXP012-30QLJ, U1 LTC4412xS6, U2 LTC4412xS6

Commit message: finito
Parts:
- added D1: SYS_LED, LED_SMD:LED_0603_1608Metric, symbol Device:LED
- added Q3: PXP012-30QLJ, iclr:PXP01230QLJ, symbol iclr:PXP012-30QLJ
- added Q4: FDN340P, Package_TO_SOT_SMD:SOT-23, symbol Transistor_FET:FDN340P
- added R1: 0, Resistor_SMD:R_0603_1608Metric, symbol Device:R_Small
- added R2: 10k, Resistor_SMD:R_0603_1608Metric, symbol Device:R_Small
- added R3: 470k, Resistor_SMD:R_0603_1608Metric, symbol Device:R_Small
- added R4: 3k, Resistor_SMD:R_0603_1608Metric, symbol Device:R_Small
Connections:
- net GND: now also Q4.3 (D), R2.2; no longer U1.3 (CTL)
- net at J2.1 (+), Q1.5 (D_1), Q1.6 (D_2)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: now also R1.2
- net SENSE: now reaches J3.1 (+), Q1.1 (S_1), Q1.2 (S_2), Q1.3 (S_3), U1.6 (SENSE), U2.6 (SENSE)
- net SENSE: now also Q3.5 (D_1), Q3.6 (D_2), Q3.7 (D_3), Q3.8 (D_4), Q3.9 (D_5), R3.1, R4.1; no longer Q2.1 (S_1), Q2.2 (S_2), Q2.3 (S_3)
- net STAT: now reaches U1.4 (STAT)
- net STAT: now also Q4.1 (G), R3.2
- net GATE1: now reaches Q2.4 (G), U1.5 (GATE)
- net GATE1: now also Q3.4 (G)
- new net: Q2.1 (S_1), Q2.2 (S_2), Q2.3 (S_3), Q3.1 (S_1), Q3.2 (S_2), Q3.3 (S_3)
- new net: D1.1 (K), Q4.2 (S)
- new net: D1.2 (A), R4.2
- new net: R1.1, R2.1, U1.3 (CTL)
- no-connect marks 2 -> 1
Other:
- note added: "BATT"
- note added: "SYS"
- moved on the sheet: H1, H2, H3, Q2
