File: DaisyChain/Connector.kicad_pcb (KiCad board)
At the start: 2 copper layers, 45 x 30 mm, 6 parts, among them J1 Conn_01x08_Female, J2 Conn_01x08_Female, J3 Conn_01x08_Female

Commit message: update
Parts:
- H1, H2: footprint MountingHole:MountingHole_3.2mm_M3_DIN965_Pad -> MountingHole:MountingHole_3.2mm_M3_DIN965
- moved H1 0.48 mm to (156.6, 96.0)
Routing:
- net /3.3V: track 57.8 -> 66.4 mm
- net /CAN-: track 40.5 -> 44.9 mm
- net /CAN+: track 43.7 -> 45.8 mm
- net GND: vias 0 -> 90
- net /DEP+: vias 0 -> 38

Commit message: silkscreen
Parts:
- added G***: LOGO, iclr:daisychain, B.Cu at (137.5, 99.5)
Other:
- board text added: "Daisy Chain"
